File: MCU Section.kicad_sch (KiCad schematic)
At the start: 69 parts, among them J4 Conn_01x04, U10 ESP32-C6-MINI-1-H8, U11 TLV62569ADRL, U12 XAL4020-222MEB, U13 GD25Q256EYIGR, U9 ESP32-P4NRW32_C22387510, X1 40MHz

Commit message: Updated the power section and battery charging IC
Parts:
- added C78: 1uF, PCM_JLCPCB:C_0402, symbol PCM_JLCPCB-Capacitors:0402,1uF
- added R42: 10kΩ, PCM_JLCPCB:R_0603, symbol PCM_JLCPCB-Resistors:0603,10kΩ
Connections:
- net C6_U0RXD: no longer U10.30 (RXD0)
- net C6_U0TXD: no longer U10.31 (TXD0)
- net ESP_3V3: now also R42.1
- net GND: now also C78.2
- net UART_TX: now reaches U9.20 (GPIO19)
- net UART_TX: now also U10.30 (RXD0)
- net UART_RX: now reaches U9.22 (GPIO20)
- net UART_RX: now also U10.31 (TXD0)
- net CHIP_PU: now reaches U9.23 (GPIO21)
- net CHIP_PU: now also U10.8 (EN), C78.1, R42.2
Other:
- note added: "UART PROTOCOL"
- note added: "~1.2V"
- moved on the sheet: C14, C15, C29, C30, C31, C32, C33, C34, C35, C36, C37, C38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

Commit message: Updated the schematic, including power section and the MCU
Parts:
- removed C32, C33, C35, C36, C39, C44, C45, C46, C48, C49, C50, C51, C52, C53, C55, C56, C57, C59, C60: 100nF, PCM_JLCPCB:C_0402, symbol PCM_JLCPCB-Capacitors:0402,100nF
- removed C37, C54: 1uF, PCM_JLCPCB:C_0402, symbol PCM_JLCPCB-Capacitors:0402,1uF
- removed C38: 10nF, PCM_JLCPCB:C_0402, symbol PCM_JLCPCB-Capacitors:0402,10nF
- removed R3: 10k, Resistor_SMD:R_0402_1005Metric, symbol Device:R_Small
- added C100, C101, C102, C103, C105, C106, C107, C108, C109, C110, C111, C112, C113, C114, C115, C116, C93, C95, C97, C99: 100nF, Capacitor_SMD:C_0201_0603Metric, symbol Device:C_Small
- added C104, C96, C98: 1uF, Capacitor_SMD:C_0201_0603Metric, symbol Device:C_Small
- added C92, C94: 10nF, Capacitor_SMD:C_0201_0603Metric, symbol Device:C_Small
- added U18, U8: ESD5451N_C2936977, ESD5451N:X1-DFN1006-2_L1.0-W0.6-P0.65-BI, symbol ESD5451N:ESD5451N_C2936977
Connections:
- net EN is gone; now on net ESP_EN: C15.1, R4.2, RST2.2
- net IO0 is gone; now on net GPIO_35: C14.1, RST1.2
- net ESP_3V3: now also C100.1, C101.1, C102.1, C109.1, C110.1, C112.1, C114.1, C115.1, C92.1, C93.1
- net ESP_VBAT: now also C116.1
- net ESP_VDD_HP: now also C111.1, C113.1, C99.1
- net GND: now also C100.2, C101.2, C102.2, C103.2, C104.2, C105.2, C106.2, C107.2, C108.2, C109.2, C110.2, C111.2, C112.2, C113.2, C114.2, C115.2, C116.2, C92.2, C93.2, C94.2, C95.2, C96.2, C97.2, C98.2, C99.2, U18.1, U8.1
- net VDDO_3: now also U9.41 (VDD_MIPI_DPHY), C107.1, C94.1, C95.1, C96.1
- net VDDO_4: now also C108.1
- net VDDO_FLASH: now also C105.1
- net VDDO_PSRAM: now also C103.1, C104.1, C106.1
- net VDD_FLASH: now also C97.1, C98.1
- net ESP_EN: now reaches U9.103 (CHIP_PU)
- net ESP_EN: now also U8.2
- net GPIO_35: now reaches U9.66 (GPIO35)
- net GPIO_35: now also U18.2
- no-connect marks 7 -> 17
Other:
- note added: "STRAPPING PINS"
- moved on the sheet: C14, C15, R4, RST1, RST2
