File: Rotary,tacts and LCD.kicad_sch (KiCad schematic)
At the start: 47 parts, among them Q1 MMBT3904, SW1 EC11E18244AU, U4 AP3032KTR-G1, U7 IS31FL3733B-QFLS4-TR

Commit message: Updated the power section and battery charging IC
Parts:
- added C66: 22nF, PCM_JLCPCB:C_0402, symbol PCM_JLCPCB-Capacitors:0402,22nF
- added C67, C68: 1uF, PCM_JLCPCB:C_0603, symbol PCM_JLCPCB-Capacitors:0603,1uF
- added C69: 10uF, PCM_JLCPCB:C_0603, symbol PCM_JLCPCB-Capacitors:0603,10uF
- added C70: 100nF, PCM_JLCPCB:C_0402, symbol PCM_JLCPCB-Capacitors:0402,100nF
- added U14: RT9193-18GB, RT9193-18GB:SOT-23-5_L3.0-W1.7-P0.95-LS2.8-BR, symbol RT9193-18GB:RT9193-18GB
Connections:
- net Core_5V: now also C68.1, U14.1 (VIN), U14.3 (EN)
- net ESP_3V3: now also C69.1, C70.1
- net GND: now also C66.2, C67.2, C68.2, C69.2, C70.2, U14.2 (GND)
- net VCC_1.8V: now also C67.1, U14.5 (VOUT)
- new net: C66.1, U14.4 (BP)
Other:
- note added: "1.8V LDO"
- moved on the sheet: MX31, S1
